Commit message: Add project docs and clean repo config

File: Mini_Dog_URDF_description/urdf/Mini_Dog_URDF.xacro (robot description, xacro)
@@ -4,5 +4,4 @@
 <xacro:include filename="$(find Mini_Dog_URDF_description)/urdf/ros2_control.xacro" />
 <xacro:include filename="$(find Mini_Dog_URDF_description)/urdf/Mini_Dog_URDF.gazebo" />
-<!-- Leg-to-Leg Manufacturing Asymmetry arguments -->
 <xacro:arg name="fl_damp_mult" default="1.0" />
 <xacro:arg name="rl_damp_mult" default="1.0" />
@@ -32,10 +31,4 @@
     <material name="silver" />
   </visual>
-  <collision>
-    <origin xyz="0 0 0" rpy="0 0 0" />
-    <geometry>
-      <mesh filename="package://Mini_Dog_URDF_description/meshes/base_link.stl" scale="0.001 0.001 0.001" />
-    </geometry>
-  </collision>
 </link>
 <link name="Femur_left_1">
@@ -43,5 +36,5 @@
     <origin xyz="-0.010006923148837377 -0.01366093016271058 -0.001499999999999991" rpy="0 0 0" />
     <mass value="0.0018979345824833387" />
-    <inertia ixx="2.729e-07" ixy="-1.460e-07" ixz="0.0" iyy="1.202e-07" iyz="0.0" izz="3.902e-07" />
+    <inertia ixx="1e-06" ixy="-1.460e-07" ixz="0.0" iyy="1e-06" iyz="0.0" izz="1e-06" />
   </inertial>
   <visual>
@@ -52,4 +45,10 @@
     <material name="silver" />
   </visual>
+  <collision>
+    <origin xyz="0.02875 -0.0115 0.02855" rpy="0 0 0" />
+    <geometry>
+      <mesh filename="package://Mini_Dog_URDF_description/meshes/Femur_left_1.stl" scale="0.001 0.001 0.001" />
+    </geometry>
+  </collision>
 </link>
 <link name="Femur_left__1__1">
@@ -57,5 +56,5 @@
     <origin xyz="-0.010006923148837402 -0.013660930162710585 -0.0015000000000000013" rpy="0 0 0" />
     <mass value="0.0018979345824833387" />
-    <inertia ixx="2.729e-07" ixy="-1.460e-07" ixz="0.0" iyy="1.202e-07" iyz="0.0" izz="3.902e-07" />
+    <inertia ixx="1e-06" ixy="-1.460e-07" ixz="0.0" iyy="1e-06" iyz="0.0" izz="1e-06" />
   </inertial>
   <visual>
@@ -66,4 +65,10 @@
     <material name="silver" />
   </visual>
+  <collision>
+    <origin xyz="0.09125 -0.0115 0.02855" rpy="0 0 0" />
+    <geometry>
+      <mesh filename="package://Mini_Dog_URDF_description/meshes/Femur_left__1__1.stl" scale="0.001 0.001 0.001" />
+    </geometry>
+  </collision>
 </link>
 <link name="Femur_right__1__1">
@@ -71,5 +76,5 @@
     <origin xyz="-0.010006923148847043 -0.013660930162727318 0.0015000000000000083" rpy="0 0 0" />
     <mass value="0.0018979345824833387" />
-    <inertia ixx="2.729e-07" ixy="-1.460e-07" ixz="0.0" iyy="1.202e-07" iyz="0.0" izz="3.902e-07" />
+    <inertia ixx="1e-06" ixy="-1.460e-07" ixz="0.0" iyy="1e-06" iyz="0.0" izz="1e-06" />
   </inertial>
   <visual>
@@ -80,4 +85,10 @@
     <material name="silver" />
   </visual>
+  <collision>
+    <origin xyz="0.02875 -0.0115 -0.02855" rpy="0 0 0" />
+    <geometry>
+      <mesh filename="package://Mini_Dog_URDF_description/meshes/Femur_right__1__1.stl" scale="0.001 0.001 0.001" />
+    </geometry>
+  </collision>
 </link>
 <link name="Knee-bearing_1">
@@ -85,5 +96,5 @@
     <origin xyz="4.2262027211137365e-13 -1.6151621574922448e-08 0.0014999999999999979" rpy="0 0 0" />
     <mass value="0.0005654866776461869" />
-    <inertia ixx="3.252e-09" ixy="3.162e-16" ixz="0.0" iyy="3.252e-09" iyz="0.0" izz="5.655e-09" />
+    <inertia ixx="1e-06" ixy="3.162e-16" ixz="0.0" iyy="1e-06" iyz="0.0" izz="1e-06" />
   </inertial>
   <visual>
@@ -99,5 +110,5 @@
     <origin xyz="4.2261333321746974e-13 -1.6151621543697425e-08 0.0015000000000000083" rpy="0 0 0" />
     <mass value="0.0005654866776461869" />
-    <inertia ixx="3.252e-09" ixy="3.162e-16" ixz="0.0" iyy="3.252e-09" iyz="0.0" izz="5.655e-09" />
+    <inertia ixx="1e-06" ixy="3.162e-16" ixz="0.0" iyy="1e-06" iyz="0.0" izz="1e-06" />
   </inertial>
   <visual>
@@ -113,5 +124,5 @@
     <origin xyz="4.2264108879308537e-13 -1.6151621533289084e-08 -0.0014999999999999944" rpy="0 0 0" />
     <mass value="0.0005654866776461869" />
-    <inertia ixx="3.252e-09" ixy="3.162e-16" ixz="0.0" iyy="3.252e-09" iyz="0.0" izz="5.655e-09" />
+    <inertia ixx="1e-06" ixy="3.162e-16" ixz="0.0" iyy="1e-06" iyz="0.0" izz="1e-06" />
   </inertial>
   <visual>
@@ -127,5 +138,5 @@
     <origin xyz="4.22592516535758e-13 -1.6151621522880744e-08 -0.0014999999999999944" rpy="0 0 0" />
     <mass value="0.0005654866776461869" />
-    <inertia ixx="3.252e-09" ixy="3.162e-16" ixz="0.0" iyy="3.252e-09" iyz="0.0" izz="5.655e-09" />
+    <inertia ixx="1e-06" ixy="3.162e-16" ixz="0.0" iyy="1e-06" iyz="0.0" izz="1e-06" />
   </inertial>
   <visual>
@@ -141,5 +152,5 @@
     <origin xyz="-0.010006923148847102 -0.01366093016272731 0.0015000000000000083" rpy="0 0 0" />
     <mass value="0.0018979345824833387" />
-    <inertia ixx="2.729e-07" ixy="-1.460e-07" ixz="0.0" iyy="1.202e-07" iyz="0.0" izz="3.902e-07" />
+    <inertia ixx="1e-06" ixy="-1.460e-07" ixz="0.0" iyy="1e-06" iyz="0.0" izz="1e-06" />
   </inertial>
   <visual>
@@ -150,4 +161,10 @@
     <material name="silver" />
   </visual>
+  <collision>
+    <origin xyz="0.09115 -0.0115 -0.02855" rpy="0 0 0" />
+    <geometry>
+      <mesh filename="package://Mini_Dog_URDF_description/meshes/Femur_right_1.stl" scale="0.001 0.001 0.001" />
+    </geometry>
+  </collision>
 </link>
 <link name="PTK_7465_v3_1">
@@ -155,5 +172,5 @@
     <origin xyz="0.013901343647080108 4.614364446098307e-16 0.005774925332524017" rpy="0 0 0" />
     <mass value="0.013830683338000317" />
-    <inertia ixx="8.651e-07" ixy="7.003e-18" ixz="8.092e-08" iyy="1.384e-06" iyz="0.0" izz="8.269e-07" />
+    <inertia ixx="1e-06" ixy="7.003e-18" ixz="8.092e-08" iyy="1.384e-06" iyz="0.0" izz="1e-06" />
   </inertial>
   <visual>
@@ -175,5 +192,5 @@
     <origin xyz="-0.013901343647080094 -4.666406150377611e-16 0.005774925332524007" rpy="0 0 0" />
     <mass value="0.013830683338000317" />
-    <inertia ixx="8.651e-07" ixy="7.003e-18" ixz="8.092e-08" iyy="1.384e-06" iyz="0.0" izz="8.269e-07" />
+    <inertia ixx="1e-06" ixy="7.003e-18" ixz="8.092e-08" iyy="1.384e-06" iyz="0.0" izz="1e-06" />
   </inertial>
   <visual>
@@ -195,5 +212,5 @@
     <origin xyz="0.013901343647080122 -4.562322741819003e-16 -0.005774925332524003" rpy="0 0 0" />
     <mass value="0.013830683338000317" />
-    <inertia ixx="8.651e-07" ixy="7.003e-18" ixz="8.092e-08" iyy="1.384e-06" iyz="0.0" izz="8.269e-07" />
+    <inertia ixx="1e-06" ixy="7.003e-18" ixz="8.092e-08" iyy="1.384e-06" iyz="0.0" izz="1e-06" />
   </inertial>
   <visual>
@@ -215,5 +232,5 @@
     <origin xyz="0.013098656352919888 4.753142324176451e-16 -0.005774925332524003" rpy="0 0 0" />
     <mass value="0.013830683338000317" />
-    <inertia ixx="8.651e-07" ixy="7.003e-18" ixz="8.092e-08" iyy="1.384e-06" iyz="0.0" izz="8.269e-07" />
+    <inertia ixx="1e-06" ixy="7.003e-18" ixz="8.092e-08" iyy="1.384e-06" iyz="0.0" izz="1e-06" />
   </inertial>
   <visual>
@@ -244,10 +261,4 @@
     <material name="silver" />
   </visual>
-  <collision>
-    <origin xyz="0.0125 -0.02 -0.0" rpy="0 0 0" />
-    <geometry>
-      <mesh filename="package://Mini_Dog_URDF_description/meshes/Esp32_Platform_1.stl" scale="0.001 0.001 0.001" />
-    </geometry>
-  </collision>
 </link>
 <link name="Battery-Platform_1">
@@ -255,5 +266,5 @@
     <origin xyz="-0.04839459526795026 0.008456964256046237 2.4369884796728917e-07" rpy="0 0 0" />
     <mass value="0.02968226258570684" />
-    <inertia ixx="9.496e-06" ixy="-9.220e-08" ixz="-3.500e-10" iyy="3.870e-05" iyz="2.500e-11" izz="3.009e-05" />
+    <inertia ixx="9.496e-06" ixy="-9.220e-08" ixz="-3.500e-10" iyy="3.87e-05" iyz="2.500e-11" izz="3.009e-05" />
   </inertial>
   <visual>
@@ -264,10 +275,4 @@
     <material name="silver" />
   </visual>
-  <collision>
-    <origin xyz="0.0125 -0.025 -0.0" rpy="0 0 0" />
-    <geometry>
-      <mesh filename="package://Mini_Dog_URDF_description/meshes/Battery-Platform_1.stl" scale="0.001 0.001 0.001" />
-    </geometry>
-  </collision>
 </link>
 <link name="Head_1">
@@ -275,5 +280,5 @@
     <origin xyz="-0.047442416576135266 0.011157188276318758 -3.895671952087887e-07" rpy="0 0 0" />
     <mass value="0.03652813810083239" />
-    <inertia ixx="1.310e-05" ixy="-1.127e-08" ixz="-7.210e-09" iyy="5.162e-05" iyz="7.700e-11" izz="4.078e-05" />
+    <inertia ixx="1.31e-05" ixy="-1.127e-08" ixz="-7.210e-09" iyy="5.162e-05" iyz="7.700e-11" izz="4.078e-05" />
   </inertial>
   <visual>
@@ -284,16 +289,10 @@
     <material name="silver" />
   </visual>
-  <collision>
-    <origin xyz="0.0125 -0.038 -0.0" rpy="0 0 0" />
-    <geometry>
-      <mesh filename="package://Mini_Dog_URDF_description/meshes/Head_1.stl" scale="0.001 0.001 0.001" />
-    </geometry>
-  </collision>
 </link>
 <link name="Servo_Horn_1">
   <inertial>
     <origin xyz="-0.005385823895367976 0.003109506875798666 -0.000899999999999998" rpy="0 0 0" />
-    <mass value="0.0003000218571105137" />
-    <inertia ixx="4.152e-09" ixy="3.561e-09" ixz="0.0" iyy="8.264e-09" iyz="0.0" izz="1.225e-08" />
+    <mass value="0.00600044" />
+    <inertia ixx="1e-06" ixy="3.561e-09" ixz="0.0" iyy="1e-06" iyz="0.0" izz="1e-06" />
   </inertial>
   <visual>
@@ -308,6 +307,6 @@
   <inertial>
     <origin xyz="-0.005385823895368014 0.003109506875798628 -0.0008999999999999946" rpy="0 0 0" />
-    <mass value="0.0003000218571105137" />
-    <inertia ixx="4.152e-09" ixy="3.561e-09" ixz="0.0" iyy="8.264e-09" iyz="0.0" izz="1.225e-08" />
+    <mass value="0.00600044" />
+    <inertia ixx="1e-06" ixy="3.561e-09" ixz="0.0" iyy="1e-06" iyz="0.0" izz="1e-06" />
   </inertial>
   <visual>
@@ -322,6 +321,6 @@
   <inertial>
     <origin xyz="-0.0053858238953680415 0.0031095068757986417 0.0008999999999999876" rpy="0 0 0" />
-    <mass value="0.0003000218571105137" />
-    <inertia ixx="4.152e-09" ixy="3.561e-09" ixz="0.0" iyy="8.264e-09" iyz="0.0" izz="1.225e-08" />
+    <mass value="0.00600044" />
+    <inertia ixx="1e-06" ixy="3.561e-09" ixz="0.0" iyy="1e-06" iyz="0.0" izz="1e-06" />
   </inertial>
   <visual>
@@ -336,6 +335,6 @@
   <inertial>
     <origin xyz="-0.005385823895367969 0.00310950687579864 0.0009000000000000154" rpy="0 0 0" />
-    <mass value="0.0003000218571105137" />
-    <inertia ixx="4.152e-09" ixy="3.561e-09" ixz="0.0" iyy="8.264e-09" iyz="0.0" izz="1.225e-08" />
+    <mass value="0.00600044" />
+    <inertia ixx="1e-06" ixy="3.561e-09" ixz="0.0" iyy="1e-06" iyz="0.0" izz="1e-06" />
   </inertial>
   <visual>
@@ -351,5 +350,5 @@
     <origin xyz="0.006315466034834807 -0.00700471170764588 -0.00400034052338508" rpy="0 0 0" />
     <mass value="0.0012633506773960263" />
-    <inertia ixx="1.371e-07" ixy="1.261e-07" ixz="1.022e-08" iyy="1.437e-07" iyz="-7.896e-09" izz="2.706e-07" />
+    <inertia ixx="1e-06" ixy="1.261e-07" ixz="1.022e-08" iyy="1e-06" iyz="-7.896e-09" izz="1e-06" />
   </inertial>
   <visual>
@@ -360,4 +359,10 @@
     <material name="silver" />
   </visual>
+  <collision>
+    <origin xyz="0.04875 0.023141 -0.03155" rpy="0 0 0" />
+    <geometry>
+      <mesh filename="package://Mini_Dog_URDF_description/meshes/Tibia_right_1.stl" scale="0.001 0.001 0.001" />
+    </geometry>
+  </collision>
 </link>
 <link name="Tibia_right__1__1">
@@ -365,5 +370,5 @@
     <origin xyz="0.0063154660348347935 -0.007004711707645817 -0.004000340523385073" rpy="0 0 0" />
     <mass value="0.0012633506773960263" />
-    <inertia ixx="1.371e-07" ixy="1.261e-07" ixz="1.022e-08" iyy="1.437e-07" iyz="-7.896e-09" izz="2.706e-07" />
+    <inertia ixx="1e-06" ixy="1.261e-07" ixz="1.022e-08" iyy="1e-06" iyz="-7.896e-09" izz="1e-06" />
   </inertial>
   <visual>
@@ -374,4 +379,10 @@
     <material name="silver" />
   </visual>
+  <collision>
+    <origin xyz="0.11115 0.023141 -0.03155" rpy="0 0 0" />
+    <geometry>
+      <mesh filename="package://Mini_Dog_URDF_description/meshes/Tibia_right__1__1.stl" scale="0.001 0.001 0.001" />
+    </geometry>
+  </collision>
 </link>
 <link name="Tibia_left_1">
@@ -379,5 +390,5 @@
     <origin xyz="0.006333544782987942 -0.007024764284155865 0.0040174405387894616" rpy="0 0 0" />
     <mass value="0.001259743842688641" />
-    <inertia ixx="1.371e-07" ixy="1.261e-07" ixz="1.022e-08" iyy="1.437e-07" iyz="-7.896e-09" izz="2.706e-07" />
+    <inertia ixx="1e-06" ixy="1.261e-07" ixz="1.022e-08" iyy="1e-06" iyz="-7.896e-09" izz="1e-06" />
   </inertial>
   <visual>
@@ -388,4 +399,10 @@
     <material name="silver" />
   </visual>
+  <collision>
+    <origin xyz="0.04875 0.023141 0.03155" rpy="0 0 0" />
+    <geometry>
+      <mesh filename="package://Mini_Dog_URDF_description/meshes/Tibia_left_1.stl" scale="0.001 0.001 0.001" />
+    </geometry>
+  </collision>
 </link>
 <link name="Tibia_left__1__1">
@@ -393,5 +410,5 @@
     <origin xyz="0.006333544782987935 -0.007024764284155865 0.004017440538789451" rpy="0 0 0" />
     <mass value="0.001259743842688641" />
-    <inertia ixx="1.371e-07" ixy="1.261e-07" ixz="1.022e-08" iyy="1.437e-07" iyz="-7.896e-09" izz="2.706e-07" />
+    <inertia ixx="1e-06" ixy="1.261e-07" ixz="1.022e-08" iyy="1e-06" iyz="-7.896e-09" izz="1e-06" />
   </inertial>
   <visual>
@@ -402,82 +419,8 @@
     <material name="silver" />
   </visual>
-</link>
-<link name="Foot_1">
-  <inertial>
-    <origin xyz="0.0010517312581306316 -0.0035929376359565487 -2.462578752027156e-13" rpy="0 0 0" />
-    <mass value="0.00017266714486627533" />
-    <inertia ixx="1.091e-09" ixy="4.700e-11" ixz="0.0" iyy="9.440e-10" iyz="0.0" izz="1.105e-09" />
-  </inertial>
-  <visual>
-    <origin xyz="0.023405 0.05387 0.02685" rpy="0 0 0" />
-    <geometry>
-      <mesh filename="package://Mini_Dog_URDF_description/meshes/Foot_1.stl" scale="0.001 0.001 0.001" />
-    </geometry>
-    <material name="silver" />
-  </visual>
-  <collision>
-    <origin xyz="0.00087 0.00767 0" rpy="0 0 0" />
-    <geometry>
-      <sphere radius="0.015" />
-    </geometry>
-  </collision>
-</link>
-<link name="Foot__3__1">
-  <inertial>
-    <origin xyz="0.0010517312581306872 -0.0035929376359565557 -2.4625440575576363e-13" rpy="0 0 0" />
-    <mass value="0.00017266714486627533" />
-    <inertia ixx="1.091e-09" ixy="4.700e-11" ixz="0.0" iyy="9.440e-10" iyz="0.0" izz="1.105e-09" />
-  </inertial>
-  <visual>
-    <origin xyz="0.023405 0.05387 -0.02685" rpy="0 0 0" />
-    <geometry>
-      <mesh filename="package://Mini_Dog_URDF_description/meshes/Foot__3__1.stl" scale="0.001 0.001 0.001" />
-    </geometry>
-    <material name="silver" />
-  </visual>
-  <collision>
-    <origin xyz="0.00087 0.00767 0" rpy="0 0 0" />
-    <geometry>
-      <sphere radius="0.015" />
-    </geometry>
-  </collision>
-</link>
-<link name="Foot__1__1">
-  <inertial>
-    <origin xyz="0.001051731258130656 -0.0035929376359565 -2.4625093630881167e-13" rpy="0 0 0" />
-    <mass value="0.00017266714486627533" />
-    <inertia ixx="1.091e-09" ixy="4.700e-11" ixz="0.0" iyy="9.440e-10" iyz="0.0" izz="1.105e-09" />
-  </inertial>
-  <visual>
-    <origin xyz="0.085805 0.05387 -0.02685" rpy="0 0 0" />
-    <geometry>
-      <mesh filename="package://Mini_Dog_URDF_description/meshes/Foot__1__1.stl" scale="0.001 0.001 0.001" />
-    </geometry>
-    <material name="silver" />
-  </visual>
-  <collision>
-    <origin xyz="0.00087 0.00767 0" rpy="0 0 0" />
-    <geometry>
-      <sphere radius="0.015" />
-    </geometry>
-  </collision>
-</link>
-<link name="Foot__2__1">
-  <inertial>
-    <origin xyz="0.0010517312581306143 -0.0035929376359565626 -2.4626828354357144e-13" rpy="0 0 0" />
-    <mass value="0.00017266714486627533" />
-    <inertia ixx="1.091e-09" ixy="4.700e-11" ixz="0.0" iyy="9.440e-10" iyz="0.0" izz="1.105e-09" />
-  </inertial>
-  <visual>
-    <origin xyz="0.085905 0.05387 0.02685" rpy="0 0 0" />
-    <geometry>
-      <mesh filename="package://Mini_Dog_URDF_description/meshes/Foot__2__1.stl" scale="0.001 0.001 0.001" />
-    </geometry>
-    <material name="silver" />
-  </visual>
-  <collision>
-    <origin xyz="0.00087 0.00767 0" rpy="0 0 0" />
-    <geometry>
-      <sphere radius="0.015" />
+  <collision>
+    <origin xyz="0.11125 0.023141 0.03155" rpy="0 0 0" />
+    <geometry>
+      <mesh filename="package://Mini_Dog_URDF_description/meshes/Tibia_left__1__1.stl" scale="0.001 0.001 0.001" />
     </geometry>
   </collision>
@@ -486,6 +429,6 @@
   <inertial>
     <origin xyz="0.0081584319459116 0.017495030023254827 0.0015000000000000013" rpy="0 0 0" />
-    <mass value="0.0007024792263066811" />
-    <inertia ixx="9.632e-08" ixy="-4.381e-08" ixz="0.0" iyy="2.280e-08" iyz="0.0" izz="1.181e-07" />
+    <mass value="0.0140496" />
+    <inertia ixx="1.9264e-06" ixy="-4.381e-08" ixz="0.0" iyy="1e-06" iyz="0.0" izz="2.362e-06" />
   </inertial>
   <visual>
@@ -500,6 +443,6 @@
   <inertial>
     <origin xyz="0.008158431945911593 0.017495030023254816 0.0015000000000000013" rpy="0 0 0" />
-    <mass value="0.0007024792263066811" />
-    <inertia ixx="9.632e-08" ixy="-4.381e-08" ixz="0.0" iyy="2.280e-08" iyz="0.0" izz="1.181e-07" />
+    <mass value="0.0140496" />
+    <inertia ixx="1.9264e-06" ixy="-4.381e-08" ixz="0.0" iyy="1e-06" iyz="0.0" izz="2.362e-06" />
   </inertial>
   <visual>
@@ -514,6 +457,6 @@
   <inertial>
     <origin xyz="0.008158431945911641 0.017495030023254823 -0.0014999999999999875" rpy="0 0 0" />
-    <mass value="0.0007024792263066811" />
-    <inertia ixx="9.632e-08" ixy="-4.381e-08" ixz="0.0" iyy="2.280e-08" iyz="0.0" izz="1.181e-07" />
+    <mass value="0.0140496" />
+    <inertia ixx="1.9264e-06" ixy="-4.381e-08" ixz="0.0" iyy="1e-06" iyz="0.0" izz="2.362e-06" />
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