Commit message: Update project files

File: Mini_Dog_URDF_description/urdf/Mini_Dog_URDF.xacro (robot description, xacro)
@@ -45,10 +45,4 @@
     <material name="silver" />
   </visual>
-  <collision>
-    <origin xyz="0.02875 -0.0115 0.02855" rpy="0 0 0" />
-    <geometry>
-      <mesh filename="package://Mini_Dog_URDF_description/meshes/Femur_left_1.stl" scale="0.001 0.001 0.001" />
-    </geometry>
-  </collision>
 </link>
 <link name="Femur_left__1__1">
@@ -65,10 +59,4 @@
     <material name="silver" />
   </visual>
-  <collision>
-    <origin xyz="0.09125 -0.0115 0.02855" rpy="0 0 0" />
-    <geometry>
-      <mesh filename="package://Mini_Dog_URDF_description/meshes/Femur_left__1__1.stl" scale="0.001 0.001 0.001" />
-    </geometry>
-  </collision>
 </link>
 <link name="Femur_right__1__1">
@@ -85,10 +73,4 @@
     <material name="silver" />
   </visual>
-  <collision>
-    <origin xyz="0.02875 -0.0115 -0.02855" rpy="0 0 0" />
-    <geometry>
-      <mesh filename="package://Mini_Dog_URDF_description/meshes/Femur_right__1__1.stl" scale="0.001 0.001 0.001" />
-    </geometry>
-  </collision>
 </link>
 <link name="Knee-bearing_1">
@@ -161,10 +143,4 @@
     <material name="silver" />
   </visual>
-  <collision>
-    <origin xyz="0.09115 -0.0115 -0.02855" rpy="0 0 0" />
-    <geometry>
-      <mesh filename="package://Mini_Dog_URDF_description/meshes/Femur_right_1.stl" scale="0.001 0.001 0.001" />
-    </geometry>
-  </collision>
 </link>
 <link name="PTK_7465_v3_1">
@@ -181,10 +157,4 @@
     <material name="silver" />
   </visual>
-  <collision>
-    <origin xyz="0.04795 -0.0115 0.02" rpy="0 0 0" />
-    <geometry>
-      <mesh filename="package://Mini_Dog_URDF_description/meshes/PTK_7465_v3_1.stl" scale="0.001 0.001 0.001" />
-    </geometry>
-  </collision>
 </link>
 <link name="PTK_7465_v3__1___1__1">
@@ -201,10 +171,4 @@
     <material name="silver" />
   </visual>
-  <collision>
-    <origin xyz="0.07205 -0.0115 0.02" rpy="0 0 0" />
-    <geometry>
-      <mesh filename="package://Mini_Dog_URDF_description/meshes/PTK_7465_v3__1___1__1.stl" scale="0.001 0.001 0.001" />
-    </geometry>
-  </collision>
 </link>
 <link name="PTK_7465_v3__1__1">
@@ -221,10 +185,4 @@
     <material name="silver" />
   </visual>
-  <collision>
-    <origin xyz="0.04795 -0.0115 -0.02" rpy="0 0 0" />
-    <geometry>
-      <mesh filename="package://Mini_Dog_URDF_description/meshes/PTK_7465_v3__1__1.stl" scale="0.001 0.001 0.001" />
-    </geometry>
-  </collision>
 </link>
 <link name="PTK_7465_v3__1___1___1__1">
@@ -241,10 +199,4 @@
     <material name="silver" />
   </visual>
-  <collision>
-    <origin xyz="0.09895 -0.0115 -0.02" rpy="0 0 0" />
-    <geometry>
-      <mesh filename="package://Mini_Dog_URDF_description/meshes/PTK_7465_v3__1___1___1__1.stl" scale="0.001 0.001 0.001" />
-    </geometry>
-  </collision>
 </link>
 <link name="Esp32_Platform_1">
@@ -359,10 +311,4 @@
     <material name="silver" />
   </visual>
-  <collision>
-    <origin xyz="0.04875 0.023141 -0.03155" rpy="0 0 0" />
-    <geometry>
-      <mesh filename="package://Mini_Dog_URDF_description/meshes/Tibia_right_1.stl" scale="0.001 0.001 0.001" />
-    </geometry>
-  </collision>
 </link>
 <link name="Tibia_right__1__1">
@@ -379,10 +325,4 @@
     <material name="silver" />
   </visual>
-  <collision>
-    <origin xyz="0.11115 0.023141 -0.03155" rpy="0 0 0" />
-    <geometry>
-      <mesh filename="package://Mini_Dog_URDF_description/meshes/Tibia_right__1__1.stl" scale="0.001 0.001 0.001" />
-    </geometry>
-  </collision>
 </link>
 <link name="Tibia_left_1">
@@ -399,10 +339,4 @@
     <material name="silver" />
   </visual>
-  <collision>
-    <origin xyz="0.04875 0.023141 0.03155" rpy="0 0 0" />
-    <geometry>
-      <mesh filename="package://Mini_Dog_URDF_description/meshes/Tibia_left_1.stl" scale="0.001 0.001 0.001" />
-    </geometry>
-  </collision>
 </link>
 <link name="Tibia_left__1__1">
@@ -419,10 +353,4 @@
     <material name="silver" />
   </visual>
-  <collision>
-    <origin xyz="0.11125 0.023141 0.03155" rpy="0 0 0" />
-    <geometry>
-      <mesh filename="package://Mini_Dog_URDF_description/meshes/Tibia_left__1__1.stl" scale="0.001 0.001 0.001" />
-    </geometry>
-  </collision>
 </link>
 <link name="Pushrod_1">
@@ -702,10 +630,4 @@
       <material name="silver" />
     </visual>
-  <collision>
-      <origin rpy="0 0 0" xyz="0.024454 0.052063 0.02555" />
-      <geometry>
-        <mesh filename="package://Mini_Dog_URDF_description/meshes/Foot_Bearing_holder_1.stl" scale="0.001 0.001 0.001" />
-      </geometry>
-    </collision>
   </link>
   <link name="Foot_Bearing_holder__1__1">
@@ -722,10 +644,4 @@
       <material name="silver" />
     </visual>
-  <collision>
-      <origin rpy="0 0 0" xyz="0.024743 0.051076 -0.02555" />
-      <geometry>
-        <mesh filename="package://Mini_Dog_URDF_description/meshes/Foot_Bearing_holder__1__1.stl" scale="0.001 0.001 0.001" />
-      </geometry>
-    </collision>
   </link>
   <link name="Foot_Bearing_holder__3__1">
@@ -742,10 +658,4 @@
       <material name="silver" />
     </visual>
-  <collision>
-      <origin rpy="0 0 0" xyz="0.087243 0.051076 0.02855" />
-      <geometry>
-        <mesh filename="package://Mini_Dog_URDF_description/meshes/Foot_Bearing_holder__3__1.stl" scale="0.001 0.001 0.001" />
-      </geometry>
-    </collision>
   </link>
   <link name="Foot_Bearing_holder__2__1">
@@ -762,10 +672,4 @@
       <material name="silver" />
     </visual>
-  <collision>
-      <origin rpy="0 0 0" xyz="0.087143 0.051076 -0.02555" />
-      <geometry>
-        <mesh filename="package://Mini_Dog_URDF_description/meshes/Foot_Bearing_holder__2__1.stl" scale="0.001 0.001 0.001" />
-      </geometry>
-    </collision>
   </link>
   <link name="FootWheel_Ratchet_1">
@@ -783,7 +687,7 @@
     </visual>
     <collision>
-      <origin rpy="1.5708 0 0" xyz="0.0 0.0 0.0015" />
-      <geometry>
-        <cylinder length="0.003" radius="0.008" />
+      <origin xyz="0.0 0.0 0.0" rpy="0 0 0" />
+      <geometry>
+        <sphere radius="0.015"/>
       </geometry>
     </collision>
@@ -803,7 +707,7 @@
     </visual>
     <collision>
-      <origin rpy="1.5708 0 0" xyz="0.0 0.0 -0.0015" />
-      <geometry>
-        <cylinder length="0.003" radius="0.008" />
+      <origin xyz="0.0 0.0 0.0" rpy="0 0 0" />
+      <geometry>
+        <sphere radius="0.015"/>
       </geometry>
     </collision>
@@ -823,7 +727,7 @@
     </visual>
     <collision>
-      <origin rpy="1.5708 0 0" xyz="0.0 0.0 -0.0015" />
-      <geometry>
-        <cylinder length="0.003" radius="0.008" />
+      <origin xyz="0.0 0.0 0.0" rpy="0 0 0" />
+      <geometry>
+        <sphere radius="0.015"/>
       </geometry>
     </collision>
@@ -843,7 +747,7 @@
     </visual>
     <collision>
-      <origin rpy="1.5708 0 0" xyz="0.0 0.0 -0.0015" />
-      <geometry>
-        <cylinder length="0.003" radius="0.008" />
+      <origin xyz="0.0 0.0 0.0" rpy="0 0 0" />
+      <geometry>
+        <sphere radius="0.015"/>
       </geometry>
     </collision>
@@ -863,7 +767,7 @@
     </visual>
     <collision>
-      <origin rpy="0 0 0" xyz="0.0 -0.001 0.0" />
-      <geometry>
-        <sphere radius="0.008" />
+      <origin xyz="0.0 0.0 0.0" rpy="0 0 0" />
+      <geometry>
+        <sphere radius="0.015"/>
       </geometry>
     </collision>
@@ -883,7 +787,7 @@
     </visual>
     <collision>
-      <origin rpy="0 0 0" xyz="0.0 -0.001 0.0" />
-      <geometry>
-        <sphere radius="0.008" />
+      <origin xyz="0.0 0.0 0.0" rpy="0 0 0" />
+      <geometry>
+        <sphere radius="0.015"/>
       </geometry>
     </collision>
@@ -903,7 +807,7 @@
     </visual>
     <collision>
-      <origin rpy="0 0 0" xyz="0.0 -0.001 0.0" />
-      <geometry>
-        <sphere radius="0.008" />
+      <origin xyz="0.0 0.0 0.0" rpy="0 0 0" />
+      <geometry>
+        <sphere radius="0.015"/>
       </geometry>
     </collision>
@@ -923,7 +827,7 @@
     </visual>
     <collision>
-      <origin rpy="0 0 0" xyz="0.0 -0.001 0.0" />
-      <geometry>
-        <sphere radius="0.008" />
+      <origin xyz="0.0 0.0 0.0" rpy="0 0 0" />
+      <geometry>
+        <sphere radius="0.015"/>
       </geometry>
     </collision>
@@ -997,3 +901,3 @@
     <child link="Foot__3__1" />
   </joint>
-  </robot>
+</robot>
